Commit message: added payload calibration, gravity comp mode for verfication and transform from force to tool frame

File: net_ft_description/urdf/net_ft_sensor.ros2_control.xacro (robot description, xacro)
@@ -1,5 +1,5 @@
 <?xml version="1.0"?>
 <robot xmlns:xacro="http://www.ros.org/wiki/xacro">
-    <xacro:macro name="net_ft_sensor_ros2_control" params="name ip_address sensor_type rdt_sampling_rate internal_filter_rate use_hardware_biasing">
+    <xacro:macro name="net_ft_sensor_ros2_control" params="name ip_address sensor_type rdt_sampling_rate internal_filter_rate use_hardware_biasing sensor_name:=tcp_fts_sensor frame_id:=tool_link">
         <ros2_control name="${name}" type="sensor">
             <hardware>
@@ -11,5 +11,5 @@
                 <param name="use_hardware_biasing">${use_hardware_biasing}</param>
             </hardware>
-            <sensor name="tcp_fts_sensor">
+            <sensor name="${sensor_name}">
               <state_interface name="force.x"/>
               <state_interface name="force.y"/>
@@ -18,5 +18,5 @@
               <state_interface name="torque.y"/>
               <state_interface name="torque.z"/>
-              <param name="frame_id">tool_link</param>
+              <param name="frame_id">${frame_id}</param>
           </sensor>
           <gpio name="diagnostic">

File: net_ft_description/urdf/net_ft_sensor_macro.urdf.xacro (robot description, xacro)
@@ -9,5 +9,6 @@
     sensor_type
     internal_filter_rate
-    use_hardware_biasing">
+    use_hardware_biasing
+    sensor_name:=tcp_fts_sensor">
     <xacro:macro name="cylinder_inertial" params="radius length mass *origin">
       <inertial>
@@ -73,5 +74,7 @@
       rdt_sampling_rate="${rdt_sampling_rate}"
       internal_filter_rate="${internal_filter_rate}"
-      use_hardware_biasing="${use_hardware_biasing}"/>
+      use_hardware_biasing="${use_hardware_biasing}"
+      sensor_name="${sensor_name}"
+      frame_id="${prefix}fts_link"/>
   </xacro:macro>
 </robot>
