Commit message: calibration worked through many times: error did not go below residual norm of 2 N: mount checked, cable strain, different poses

File: net_ft_description/urdf/net_ft_sensor_macro.urdf.xacro (robot description, xacro)
@@ -10,5 +10,7 @@
     internal_filter_rate
     use_hardware_biasing
-    sensor_name:=tcp_fts_sensor">
+    sensor_name:=tcp_fts_sensor
+    tool_side_xyz:=''
+    tool_side_rpy:='0 0 0'">
     <xacro:macro name="cylinder_inertial" params="radius length mass *origin">
       <inertial>
@@ -64,5 +66,6 @@
       <parent link="${prefix}fts_link"/>
       <child link="${prefix}tool_mount_link"/>
-      <origin xyz="0 0 ${sensor_height}" rpy="0 0 0"/>
+      <!-- tool_side_* undo a measurement-frame correction in *origin, so the tool stays put -->
+      <origin xyz="${tool_side_xyz if tool_side_xyz else '0 0 ' + str(sensor_height)}" rpy="${tool_side_rpy}"/>
     </joint>
     <link name="${prefix}tool_mount_link"/>
